File: RP2040.kicad_sch (KiCad schematic)
At the start: 23 parts, among them J1 Conn_01x02, U7 RP2040, U8 W25Q128JVS, Y1 Crystal_GND24

Commit message: started on layout and added SD/flash/BNO
Parts:
- renumbered J1 to J2, R9 to R15, R10 to R16, R11 to R17, R12 to R18, R13 to R19, U7 to U8, U8 to U9
Connections:
- net SPI_CIPO: now reaches U8.11 (GPIO8)
- net SPI_CS_FLASH: now reaches U8.12 (GPIO9)
- net SPI_CS_SD: now reaches U8.13 (GPIO10)
- net SPI_CS_EXTRA: now reaches U8.14 (GPIO11)
- net SPI_SCK: now reaches U8.8 (GPIO6)
- net SPI_COPI: now reaches U8.9 (GPIO7)

Commit message: final
Parts:
- renumbered C19 to C12, C20 to C13, C21 to C14, C22 to C15, C23 to C16, C24 to C17, C25 to C18, C26 to C19, C27 to C20, C28 to C21, C29 to C22, C30 to C23, C31 to C24, C32 to C25, R15 to R12, R16 to R13, R17 to R14, R18 to R15, R19 to R16, U8 to U4, U9 to U5
Connections:
- net SOLENOID_2A is gone; now on net BUCK_EN_A: U4.31 (GPIO20)
- net BUCK_EN_A: no longer U4.29 (GPIO18)
- net BTN: now reaches U4.15 (GPIO12)
- net BUZZER: now reaches U4.37 (GPIO25)
- net SOLENOID_1A renamed SERVO_2A
- net SOLENOID_1B renamed SERVO_1B
- net SOLENOID_2B renamed SERVO_2B
- net SPI_CS_EXTRA renamed NEOPIXEL
- new net SERVO_1A: U4.29 (GPIO18)
- no-connect marks 0 -> 10
