File: SD.kicad_sch (KiCad schematic)
At the start: 3 parts, among them J12 Micro_SD_Card

Commit message: final
Parts:
- renumbered C38 to C31, R22 to R19
Connections:
- net GND: now also J12.9 (SHIELD)
Changed lines of the file:
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@@
+    (stroke (width 0) (type default))
+  )
+  (wire (pts (xy 160.655 106.68) (xy 160.655 106.045))
     (stroke (width 0) (type default))
   )
@@
     (stroke (width 0) (type default))
   )
+  (wire (pts (xy 160.655 106.045) (xy 160.02 106.045))
+    (stroke (width 0) (type default))
+  )
   (wire (pts (xy 115.57 88.265) (xy 116.84 88.265))
     (stroke (width 0) (type default))
@@
     (effects (font (size 1.27 1.27)) (justify right))
   )
+  (symbol (lib_id "power:GND") (at 160.655 106.68 0) (unit 1)
+    (in_bom yes) (on_board yes) (dnp no) (fields_autoplaced)
+    (property "Reference" "#PWR059" (at 160.655 113.03 0)
+      (effects (font (size 1.27 1.27)) hide)
+    )
+    (property "Value" "GND" (at 160.655 111.125 0)
+      (effects (font (size 1.27 1.27)))
+    )
+    (property "Footprint" "" (at 160.655 106.68 0)
+      (effects (font (size 1.27 1.27)) hide)
+    )
+    (property "Datasheet" "" (at 160.655 106.68 0)
+      (effects (font (size 1.27 1.27)) hide)
+    )
+    (pin "1")
+    (instances
+      (project "UMRT_FC_R2"
+        (path "/27c40824-3c02-48dc-87e8-ac576671a38f/92580f07-8c4c-4842-873e-67db8948eb3d"
+          (reference "#PWR059") (unit 1)
+        )
+      )
+    )
+  )
   (symbol (lib_id "power:+3V3") (at 108.585 76.835 0) (unit 1)
     (in_bom yes) (on_board yes) (dnp no) (fields_autoplaced)
-    (property "Reference" "#PWR059" (at 108.585 80.645 0)
+    (property "Reference" "#PWR058" (at 108.585 80.645 0)
       (effects (font (size 1.27 1.27)) hide)
     )
@@
     (pin "1")
     (instances
-      (project "UMRT_FC_R1"
-        (path "/27c40824-3c02-48dc-87e8-ac576671a38f/92580f07-8c4c-4842-873e-67db8948eb3d"
-          (reference "#PWR059") (unit 1)
+      (project "UMRT_FC_R2"
+        (path "/27c40824-3c02-48dc-87e8-ac576671a38f/92580f07-8c4c-4842-873e-67db8948eb3d"
+          (reference "#PWR058") (unit 1)
         )
       )
@@
   (symbol (lib_id "Device:R_Small") (at 108.585 80.645 0) (unit 1)
     (in_bom yes) (on_board yes) (dnp no) (fields_autoplaced)
-    (property "Reference" "R22" (at 111.125 79.375 0)
+    (property "Reference" "R19" (at 111.125 79.375 0)
       (effects (font (size 1.27 1.27)) (justify left))
     )
@@
     (pin "2")
     (instances
-      (project "UMRT_FC_R1"
-        (path "/27c40824-3c02-48dc-87e8-ac576671a38f/92580f07-8c4c-4842-873e-67db8948eb3d"
-          (reference "R22") (unit 1)
+      (project "UMRT_FC_R2"
+        (path "/27c40824-3c02-48dc-87e8-ac576671a38f/92580f07-8c4c-4842-873e-67db8948eb3d"
+          (reference "R19") (unit 1)
         )
       )
@@
   (symbol (lib_id "power:GND") (at 92.075 97.155 0) (unit 1)
     (in_bom yes) (on_board yes) (dnp no) (fields_autoplaced)
-    (property "Reference" "#PWR058" (at 92.075 103.505 0)
+    (property "Reference" "#PWR057" (at 92.075 103.505 0)
       (effects (font (size 1.27 1.27)) hide)
     )
@@
     (pin "1")
     (instances
-      (project "UMRT_FC_R1"
-        (path "/27c40824-3c02-48dc-87e8-ac576671a38f/92580f07-8c4c-4842-873e-67db8948eb3d"
-          (reference "#PWR058") (unit 1)
+      (project "UMRT_FC_R2"
+        (path "/27c40824-3c02-48dc-87e8-ac576671a38f/92580f07-8c4c-4842-873e-67db8948eb3d"
+          (reference "#PWR057") (unit 1)
         )
       )
@@
   (symbol (lib_id "power:+3V3") (at 92.075 89.535 0) (unit 1)
     (in_bom yes) (on_board yes) (dnp no) (fields_autoplaced)
-    (property "Reference" "#PWR057" (at 92.075 93.345 0)
+    (property "Reference" "#PWR056" (at 92.075 93.345 0)
       (effects (font (size 1.27 1.27)) hide)
     )
@@
     (pin "1")
     (instances
-      (project "UMRT_FC_R1"
-        (path "/27c40824-3c02-48dc-87e8-ac576671a38f/92580f07-8c4c-4842-873e-67db8948eb3d"
-          (reference "#PWR057") (unit 1)
+      (project "UMRT_FC_R2"
+        (path "/27c40824-3c02-48dc-87e8-ac576671a38f/92580f07-8c4c-4842-873e-67db8948eb3d"
+          (reference "#PWR056") (unit 1)
         )
       )
@@
     (pin "9")
     (instances
-      (project "UMRT_FC_R1"
+      (project "UMRT_FC_R2"
         (path "/27c40824-3c02-48dc-87e8-ac576671a38f"
           (reference "J12") (unit 1)
         )
         (path "/27c40824-3c02-48dc-87e8-ac576671a38f/92580f07-8c4c-4842-873e-67db8948eb3d"
-          (reference "J12") (unit 1)
+          (reference "J13") (unit 1)
         )
       )
@@
   (symbol (lib_id "Device:C_Small") (at 92.075 93.345 0) (unit 1)
     (in_bom yes) (on_board yes) (dnp no) (fields_autoplaced)
-    (property "Reference" "C38" (at 95.25 92.0813 0)
+    (property "Reference" "C31" (at 95.25 92.0813 0)
       (effects (font (size 1.27 1.27)) (justify left))
     )
@@
     (pin "2")
     (instances
-      (project "UMRT_FC_R1"
-        (path "/27c40824-3c02-48dc-87e8-ac576671a38f/92580f07-8c4c-4842-873e-67db8948eb3d"
-          (reference "C38") (unit 1)
-        )
-      )
+      (project "UMRT_FC_R2"
+        (path "/27c40824-3c02-48dc-87e8-ac576671a38f/92580f07-8c4c-4842-873e-67db8948eb3d"
+          (reference "C31") (unit 1)
+        )
+      )
