File: UMRT_FC_R2.kicad_sch (KiCad schematic)
At the start: 8 parts, among them J1 USB_A

Commit message: final
Parts:
- added BZ1: Buzzer, Buzzer_Beeper:Buzzer_CUI_CPT-9019S-SMT, symbol Device:Buzzer
- added C1: 100n, Capacitor_SMD:C_0603_1608Metric, symbol Device:C_Small
- added D1: WS2812B, LED_SMD:LED_WS2812B_PLCC4_5.0x5.0mm_P3.2mm, symbol LED:WS2812B
- added H1, H2, H3, H4: ~, MountingHole:MountingHole_3.2mm_M3_Pad_Via, symbol Mechanical:MountingHole_Pad
- added R1: 1k, Resistor_SMD:R_0603_1608Metric, symbol Device:R_Small
- renumbered R1 to R2, R2 to R3, R3 to R4, R4 to R5, R5 to R6, R6 to R7
Connections:
- net +3V3: now also C1.1, D1.1 (VDD)
- net GND: now also BZ1.2 (+), C1.2, D1.3 (VSS), H1.1, H2.1, H3.1, H4.1, R1.1
- new net RP2040/BUZZER: BZ1.1 (-), R1.2
- new net RP2040/NEOPIXEL: D1.4 (DIN)
- no-connect marks 1 -> 2
Other:
- sheet IO ports: added S1A, S1B, S2A, S2B, SPWR_A, SPWR_B; removed S1A_N, S1A_P, S1B_N, S1B_P, S2A_N, S2A_P, S2B_N, S2B_P
- sheet RP2040 ports: added BUZZER, NEOPIXEL, SERVO_1A, SERVO_1B, SERVO_2A, SERVO_2B; removed SOLENOID_1A, SOLENOID_2A
- sheet solenoid driver A ports: added SPWR_A; removed S1A_EN, S1A_N, S1A_P, S2A_EN, S2A_N, S2A_P
- sheet solenoid driver B ports: added SPWR_B; removed S1B_EN, S1B_N, S1B_P, S2B_EN, S2B_N, S2B_P
- sheet state indication ports: added none; removed SOLENOID_1A, SOLENOID_1B, SOLENOID_2A, SOLENOID_2B
- moved on the sheet: U1
