File: flash.kicad_sch (KiCad schematic)
At the start: 3 parts, among them U10 W25Q32JVSS

Commit message: final
Parts:
- C38: footprint Capacitor_SMD:C_0402_1005Metric -> Capacitor_SMD:C_0603_1608Metric
- R19: footprint Resistor_SMD:R_0402_1005Metric -> Resistor_SMD:R_0603_1608Metric
Changed lines of the file:
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@@
     (pin "1")
     (instances
-      (project "UMRT_FC_R1"
+      (project "UMRT_FC_R2"
         (path "/27c40824-3c02-48dc-87e8-ac576671a38f"
           (reference "#PWR059") (unit 1)
@@
       (effects (font (size 1.27 1.27)) (justify left))
     )
-    (property "Footprint" "Capacitor_SMD:C_0402_1005Metric" (at 104.14 89.535 0)
+    (property "Footprint" "Capacitor_SMD:C_0603_1608Metric" (at 104.14 89.535 0)
       (effects (font (size 1.27 1.27)) hide)
     )
@@
     (pin "2")
     (instances
-      (project "UMRT_FC_R1"
+      (project "UMRT_FC_R2"
         (path "/27c40824-3c02-48dc-87e8-ac576671a38f"
           (reference "C38") (unit 1)
         )
         (path "/27c40824-3c02-48dc-87e8-ac576671a38f/e0cc0fcc-dbf5-4529-bef1-fe207310c36c"
-          (reference "C39") (unit 1)
+          (reference "C32") (unit 1)
         )
       )
@@
     (pin "8")
     (instances
-      (project "UMRT_FC_R1"
+      (project "UMRT_FC_R2"
         (path "/27c40824-3c02-48dc-87e8-ac576671a38f"
           (reference "U10") (unit 1)
         )
         (path "/27c40824-3c02-48dc-87e8-ac576671a38f/e0cc0fcc-dbf5-4529-bef1-fe207310c36c"
-          (reference "U11") (unit 1)
+          (reference "U7") (unit 1)
         )
       )
@@
     (pin "1")
     (instances
-      (project "UMRT_FC_R1"
+      (project "UMRT_FC_R2"
         (path "/27c40824-3c02-48dc-87e8-ac576671a38f"
           (reference "#PWR062") (unit 1)
@@
       (effects (font (size 1.27 1.27)) (justify left))
     )
-    (property "Footprint" "Resistor_SMD:R_0402_1005Metric" (at 111.125 91.44 0)
+    (property "Footprint" "Resistor_SMD:R_0603_1608Metric" (at 111.125 91.44 0)
       (effects (font (size 1.27 1.27)) hide)
     )
@@
     (pin "2")
     (instances
-      (project "UMRT_FC_R1"
+      (project "UMRT_FC_R2"
         (path "/27c40824-3c02-48dc-87e8-ac576671a38f"
           (reference "R19") (unit 1)
         )
         (path "/27c40824-3c02-48dc-87e8-ac576671a38f/e0cc0fcc-dbf5-4529-bef1-fe207310c36c"
-          (reference "R23") (unit 1)
+          (reference "R20") (unit 1)
         )
       )
@@
     (pin "1")
     (instances
-      (project "UMRT_FC_R1"
+      (project "UMRT_FC_R2"
         (path "/27c40824-3c02-48dc-87e8-ac576671a38f"
           (reference "#PWR060") (unit 1)
@@
     (pin "1")
     (instances
-      (project "UMRT_FC_R1"
+      (project "UMRT_FC_R2"
         (path "/27c40824-3c02-48dc-87e8-ac576671a38f"
           (reference "#PWR061") (unit 1)
