File: solenoid driver A.kicad_sch (KiCad schematic)
At the start: 19 parts

Commit message: started on layout and added SD/flash/BNO
Connections:
- net S1A_N is gone; now on net GND: D2.2 (A)
- net S2A_N is gone; now on net GND: D1.2 (A)

Commit message: final
Parts:
- removed C11, C13: 1u, Capacitor_SMD:C_0603_1608Metric, symbol Device:C_Small
- removed C12, C14: 10u, Capacitor_SMD:C_0603_1608Metric, symbol Device:C_Small
- removed D1, D2: S2JTR, Diode_SMD:D_SMB, symbol Diode:S2JTR
- removed R1, R3: 473.6, Resistor_SMD:R_0603_1608Metric, symbol Device:R_Small
- removed U3, U4: ~, Package_TO_SOT_SMD:SOT-23-6, symbol mp5036:MP5036
- C2: value 12p -> 47p
- L1: value 10u -> 6.8u
- R13: value 422 -> 158k
- R14: value 30.1 -> 30.1k
Connections:
- no-connect marks 2 -> 0
Other:
- note added: "Servo rail A"
- note removed: "Solenoid 1A"
- note removed: "Solenoid 2A"
- note removed: "Solenoid rail A"
