File: solenoid driver B.kicad_sch (KiCad schematic)
At the start: 19 parts

Commit message: started on layout and added SD/flash/BNO
Connections:
- net S1B_N is gone; now on net GND: D2.2 (A)
- net S2B_N is gone; now on net GND: D1.2 (A)
Changed lines of the file:
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@@
   (junction (at 90.17 76.2) (diameter 0) (color 0 0 0 0)
   )
+  (junction (at 165.1 74.295) (diameter 0) (color 0 0 0 0)
+  )
   (junction (at 67.31 96.52) (diameter 0) (color 0 0 0 0)
   )
   (junction (at 97.79 63.5) (diameter 0) (color 0 0 0 0)
+  )
+  (junction (at 101.6 74.295) (diameter 0) (color 0 0 0 0)
   )
   (junction (at 111.76 104.14) (diameter 0) (color 0 0 0 0)
@@
     (stroke (width 0) (type default))
   )
+  (wire (pts (xy 161.29 76.2) (xy 165.1 76.2))
+    (stroke (width 0) (type default))
+  )
   (wire (pts (xy 88.9 69.85) (xy 90.17 69.85))
     (stroke (width 0) (type default))
@@
     (stroke (width 0) (type default))
   )
+  (wire (pts (xy 165.1 76.2) (xy 165.1 74.295))
+    (stroke (width 0) (type default))
+  )
   (wire (pts (xy 97.79 69.215) (xy 97.79 76.2))
     (stroke (width 0) (type default))
@@
     (stroke (width 0) (type default))
   )
+  (wire (pts (xy 97.79 76.2) (xy 101.6 76.2))
+    (stroke (width 0) (type default))
+  )
   (wire (pts (xy 98.425 104.14) (xy 98.425 102.87))
     (stroke (width 0) (type default))
@@
   )
   (wire (pts (xy 165.1 65.405) (xy 165.1 63.5))
+    (stroke (width 0) (type default))
+  )
+  (wire (pts (xy 101.6 76.2) (xy 101.6 74.295))
     (stroke (width 0) (type default))
   )
@@
         )
         (path "/27c40824-3c02-48dc-87e8-ac576671a38f/1a09dec7-41ca-4d12-949e-139ba0104602"
-          (reference "#PWR014") (unit 1)
+          (reference "#PWR018") (unit 1)
         )
       )
@@
         )
         (path "/27c40824-3c02-48dc-87e8-ac576671a38f/1a09dec7-41ca-4d12-949e-139ba0104602"
-          (reference "#PWR019") (unit 1)
+          (reference "#PWR023") (unit 1)
         )
       )
@@
         )
         (path "/27c40824-3c02-48dc-87e8-ac576671a38f/1a09dec7-41ca-4d12-949e-139ba0104602"
-          (reference "#PWR016") (unit 1)
+          (reference "#PWR020") (unit 1)
         )
       )
@@
         )
         (path "/27c40824-3c02-48dc-87e8-ac576671a38f/1a09dec7-41ca-4d12-949e-139ba0104602"
-          (reference "R7") (unit 1)
+          (reference "R13") (unit 1)
         )
       )
@@
         )
         (path "/27c40824-3c02-48dc-87e8-ac576671a38f/1a09dec7-41ca-4d12-949e-139ba0104602"
-          (reference "U6") (unit 1)
+          (reference "U7") (unit 1)
         )
       )
@@
   (symbol (lib_id "power:+24V") (at 63.5 95.25 0) (unit 1)
     (in_bom yes) (on_board yes) (dnp no)
-    (property "Reference" "#PWR012" (at 63.5 99.06 0)
+    (property "Reference" "#PWR016" (at 63.5 99.06 0)
       (effects (font (size 1.27 1.27)) hide)
     )
@@
       (project "UMRT_FC_R1"
         (path "/27c40824-3c02-48dc-87e8-ac576671a38f/1a09dec7-41ca-4d12-949e-139ba0104602"
-          (reference "#PWR012") (unit 1)
+          (reference "#PWR016") (unit 1)
         )
       )
@@
         )
         (path "/27c40824-3c02-48dc-87e8-ac576671a38f/1a09dec7-41ca-4d12-949e-139ba0104602"
-          (reference "#PWR018") (unit 1)
+          (reference "#PWR022") (unit 1)
         )
       )
@@
         )
         (path "/27c40824-3c02-48dc-87e8-ac576671a38f/1a09dec7-41ca-4d12-949e-139ba0104602"
-          (reference "R6") (unit 1)
+          (reference "R12") (unit 1)
         )
       )
@@
         )
         (path "/27c40824-3c02-48dc-87e8-ac576671a38f/1a09dec7-41ca-4d12-949e-139ba0104602"
-          (reference "R8") (unit 1)
+          (reference "R14") (unit 1)
         )
       )
@@
         )
         (path "/27c40824-3c02-48dc-87e8-ac576671a38f/1a09dec7-41ca-4d12-949e-139ba0104602"
-          (reference "U5") (unit 1)
+          (reference "U6") (unit 1)
         )
       )
@@
         )
         (path "/27c40824-3c02-48dc-87e8-ac576671a38f/1a09dec7-41ca-4d12-949e-139ba0104602"
-          (reference "#PWR015") (unit 1)
+          (reference "#PWR019") (unit 1)
         )
       )
@@
         )
         (path "/27c40824-3c02-48dc-87e8-ac576671a38f/1a09dec7-41ca-4d12-949e-139ba0104602"
-          (reference "R5") (unit 1)
+          (reference "R11") (unit 1)
         )
       )
@@
         )
         (path "/27c40824-3c02-48dc-87e8-ac576671a38f/1a09dec7-41ca-4d12-949e-139ba0104602"
-          (reference "#PWR017") (unit 1)
+          (reference "#PWR021") (unit 1)
         )
       )
@@
         )
         (path "/27c40824-3c02-48dc-87e8-ac576671a38f/1a09dec7-41ca-4d12-949e-139ba0104602"
-          (reference "#PWR011") (unit 1)
+          (reference "#PWR015") (unit 1)
         )
       )
@@
         )
         (path "/27c40824-3c02-48dc-87e8-ac576671a38f/1a09dec7-41ca-4d12-949e-139ba0104602"
-          (reference "#PWR020") (unit 1)
+          (reference "#PWR024") (unit 1)
         )
       )
@@
         )
         (path "/27c40824-3c02-48dc-87e8-ac576671a38f/1a09dec7-41ca-4d12-949e-139ba0104602"
-          (reference "#PWR013") (unit 1)
+          (reference "#PWR017") (unit 1)
         )
       )
@@
         )
         (path "/27c40824-3c02-48dc-87e8-ac576671a38f/1a09dec7-41ca-4d12-949e-139ba0104602"
-          (reference "U4") (unit 1)
-        )
-      )
+          (reference "U5") (unit 1)
+        )
+      )

Commit message: final
Parts:
- removed C11, C13: 1u, Capacitor_SMD:C_0603_1608Metric, symbol Device:C_Small
- removed C12, C14: 10u, Capacitor_SMD:C_0603_1608Metric, symbol Device:C_Small
- removed D1, D2: S2JTR, Diode_SMD:D_SMB, symbol Diode:S2JTR
- removed R1, R3: 473.6, Resistor_SMD:R_0603_1608Metric, symbol Device:R_Small
- removed U3, U4: ~, Package_TO_SOT_SMD:SOT-23-6, symbol mp5036:MP5036
- C2: value 12p -> 47p
- L1: value 10u -> 6.8u
- R13: value 422 -> 158k
- R14: value 30.1 -> 30.1k
Connections:
- no-connect marks 2 -> 0
Other:
- note added: "Servo rail B"
- note removed: "Solenoid 1B"
- note removed: "Solenoid 2B"
- note removed: "Solenoid rail B"
