File: state indication.kicad_sch (KiCad schematic)
At the start: 18 parts

Commit message: final
Parts:
- removed D8 (x4): LED, LED_SMD:LED_0603_1608Metric, symbol Device:LED_Small
- removed R15 (x4): 5k, Resistor_SMD:R_0603_1608Metric, symbol Device:R_Small
Other:
- moved on the sheet: D8, R15
